Commit message: compiled with ros

File: gazebo/models/jackal/sensors/camera/r200.urdf.xacro (robot description, xacro)
@@ -1,5 +1,5 @@
 <?xml version="1.0"?>
 <robot name="sensor_r200" xmlns:xacro="http://ros.org/wiki/xacro">
-  <xacro:include filename="$(find oforca)/gazebo/models/jackal/sensors/camera/common_properties.urdf.xacro"/>
+  <xacro:include filename="$(find coslam)/gazebo/models/jackal/sensors/camera/common_properties.urdf.xacro"/>
   <!-- Mount and camera parameters -->
   <xacro:property name="pole_px" value="-0.103" />
@@ -34,5 +34,5 @@
        <origin xyz="${-r200_bracket_end_width/2} ${r200_bracket_end_offset_py} ${r200_bracket_end_offset_pz}" rpy="0 0 ${-M_PI/2}"/>
         <geometry>
-         <mesh filename="$(find oforca)/gazebo/models/jackal/sensors/camera/meshes/sensors/r200_bracket_end.stl" scale="0.001 0.001 0.001"/>
+         <mesh filename="$(find coslam)/gazebo/models/jackal/sensors/camera/meshes/sensors/r200_bracket_end.stl" scale="0.001 0.001 0.001"/>
         </geometry>
         <xacro:insert_block name="material_dark_grey" />
@@ -49,5 +49,5 @@
        <origin xyz="0 0 0" rpy="0 0 ${M_PI/2}"/>
         <geometry>
-         <mesh filename="$(find oforca)/gazebo/models/jackal/sensors/camera/meshes/sensors/r200_bracket.stl" scale="0.001 0.001 0.001"/>
+         <mesh filename="$(find coslam)/gazebo/models/jackal/sensors/camera/meshes/sensors/r200_bracket.stl" scale="0.001 0.001 0.001"/>
         </geometry>
         <xacro:insert_block name="material_dark_grey" />
@@ -64,5 +64,5 @@
        <origin xyz="${r200_bracket_end_width/2} 0 ${-r200_bracket_end_offset_pz}" rpy="0 0 ${M_PI/2}"/>
         <geometry>
-         <mesh filename="$(find oforca)/gazebo/models/jackal/sensors/camera/meshes/sensors/r200_bracket_end.stl" scale="0.001 0.001 0.001"/>
+         <mesh filename="$(find coslam)/gazebo/models/jackal/sensors/camera/meshes/sensors/r200_bracket_end.stl" scale="0.001 0.001 0.001"/>
         </geometry>
         <xacro:insert_block name="material_dark_grey" />
@@ -79,5 +79,5 @@
        <origin xyz="0 0 0" rpy="${M_PI/2} 0 ${M_PI/2}"/>
         <geometry>
-         <mesh filename="$(find oforca)/gazebo/models/jackal/sensors/camera/meshes/sensors/r200.dae" />
+         <mesh filename="$(find coslam)/gazebo/models/jackal/sensors/camera/meshes/sensors/r200.dae" />
         </geometry>
       </visual>
