Commit message: modified rgb to only one global camera

File: gazebo/models/rgbd_camera/r200.urdf.xacro (robot description, xacro)
@@ -8,5 +8,5 @@
   <link name="camera_base"/>
   <joint name="camera_base_joint" type="fixed">
-    <origin xyz="$(arg offset_px) $(arg offset_py) $(arg floor_height)" rpy="0 0 0"/>
+    <origin xyz="0 0 0" rpy="0 0 0"/>
     <parent link="camera_base"/>
     <child link="camera_base_link" />

Commit message: debugg fixing

File: gazebo/models/rgbd_camera/r200.urdf.xacro (robot description, xacro)
@@ -5,8 +5,16 @@
   <xacro:property name="r200_cam_rgb_py" value="0.018"/>
   <xacro:property name="r200_cam_rgb_pz" value="0.013"/>
-  <xacro:property name="r200_cam_depth_offset" value="0.01"/>
+  <xacro:property name="r200_cam_depth_offset" value="0.00"/>
+  <xacro:arg name="offset_pz" default="5"/>
+  <xacro:arg name="offset_r" default="0"/>
+  <xacro:arg name="offset_p" default="0"/>
+  <xacro:arg name="offset_y" default="0"/>
+  <xacro:arg name="namespace" default="rgb0"/>
+  <xacro:arg name="base_x" default="0"/>
+  <xacro:arg name="base_y" default="0"/>
+  <xacro:arg name="b_yaw" default="0"/>
   <link name="camera_base"/>
   <joint name="camera_base_joint" type="fixed">
-    <origin xyz="0 0 0" rpy="0 0 0"/>
+    <origin xyz="$(arg base_x) $(arg base_y) 0" rpy="0 0 $(arg b_yaw)"/>
     <parent link="camera_base"/>
     <child link="camera_base_link" />
@@ -60,7 +68,7 @@
     <origin xyz="${r200_cam_rgb_px} ${r200_cam_rgb_py} ${r200_cam_rgb_pz}" rpy="0 0 0"/>
     <parent link="camera_link"/>
-    <child link="camera_rgb_frame" />
+    <child link="camera_optical_frame" />
   </joint>
-  <link name="camera_rgb_frame"/>
+  <!-- <link name="camera_rgb_frame"/>
   <joint name="camera_rgb_optical_joint" type="fixed">
     <origin xyz="0 0 0" rpy="${-M_PI/2} 0 ${-M_PI/2}" />
@@ -78,8 +86,8 @@
       <origin xyz="0 0 0" rpy="${-M_PI/2} 0 ${-M_PI/2}" />
       <parent link="camera_depth_frame" />
-      <child link="camera_depth_optical_frame" />
-  </joint>
-  <link name="camera_depth_optical_frame"/>
-  <gazebo reference="camera_link">
+      <child link="camera_optical_frame" />
+  </joint> -->
+  <link name="camera_optical_frame"/>
+  <gazebo reference="camera_optical_frame">
     <sensor type="depth" name="camera">
       <always_on>true</always_on>
@@ -90,5 +98,5 @@
           <format>B8G8R8</format>
           <width>640</width>
-          <height>448</height>
+          <height>480</height>
         </image>
         <clip>
@@ -112,5 +120,5 @@
         <cameraInfoTopicName>camera_info</cameraInfoTopicName>
         <depthImageCameraInfoTopicName>depth/camera_info</depthImageCameraInfoTopicName>
-        <frameName>camera_depth_optical_frame</frameName>
+        <frameName>camera_optical_frame</frameName>
         <baseline>0.1</baseline>
         <distortion_k1>0.0</distortion_k1>
@@ -123,3 +131,20 @@
     </sensor>
   </gazebo>
+  <!-- <this one cannot be used with other velocity control> -->
+  <!-- <gazebo>
+    <plugin name="object_controller" filename="libgazebo_ros_planar_move.so">
+      <commandTopic>rgbd_cmd</commandTopic>
+      <odometryTopic>odom</odometryTopic>
+      <odometryFrame>$(arg namespace)/camera_base</odometryFrame>
+      <odometryRate>20.0</odometryRate>
+      <robotBaseFrame>odom</robotBaseFrame>
+    </plugin>
+  </gazebo>   -->
+  <!-- <gazebo>
+    <plugin name="joint_state_publisher" filename="libgazebo_ros_joint_state_publisher.so">
+       <jointName>your_joint</jointName>
+       <updateRate>50.0</updateRate>
+       <alwaysOn>true</alwaysOn>
+    </plugin>
+  </gazebo> -->
 </robot>

File: gazebo/models/robot/lightmodel.xacro (robot description, xacro)
@@ -7,7 +7,7 @@
   <xacro:property name="tag_name" value="tag36_11_00001" />
   <xacro:include filename="$(find turtlebot3_description)/urdf/common_properties.xacro"/>
-  <link name="robot_base"/>
+  <link name="base_footprint"/>
   <joint name="base_joint" type="fixed">
-    <parent link="robot_base"/>
+    <parent link="base_footprint"/>
     <child link="base_link"/>
     <origin xyz="0.0 0.0 0.010" rpy="0 0 0"/>
@@ -66,5 +66,4 @@
     <inertial>
       <origin xyz="0 0 0" />
-      <!-- <mass value="1" /> -->
       <mass value="0.005" />
       <inertia ixx="0.001" ixy="0.0" ixz="0.0"
@@ -124,5 +123,4 @@
     <inertial>
       <origin xyz="0 0 0" />
-      <!-- <mass value="1" /> -->
       <mass value="2.8498940e-02" />
       <inertia ixx="1.1175580e-05" ixy="-4.2369783e-11" ixz="-5.9381719e-09"
@@ -153,5 +151,4 @@
     <inertial>
       <origin xyz="0 0 0" />
-      <!-- <mass value="1" /> -->
       <mass value="2.8498940e-02" />
       <inertia ixx="1.1175580e-05" ixy="-4.2369783e-11" ixz="-5.9381719e-09"
@@ -167,5 +164,5 @@
       <odometrySource>world</odometrySource>
       <publishOdomTF>true</publishOdomTF>
-      <robotBaseFrame>robot_base</robotBaseFrame>
+      <robotBaseFrame>base_footprint</robotBaseFrame>
       <publishWheelTF>false</publishWheelTF>
       <publishTf>true</publishTf>
@@ -177,5 +174,5 @@
       <wheelSeparation>0.160</wheelSeparation>
       <wheelDiameter>0.066</wheelDiameter>
-      <wheelAcceleration>1</wheelAcceleration>
+      <wheelAcceleration>10</wheelAcceleration>
       <wheelTorque>10</wheelTorque>
       <rosDebugLevel>na</rosDebugLevel>
